File: _autosave-control_panel.kicad_sch (KiCad schematic)
At the start: 17 parts, among them J3 PJ301M-12, J4 PJ301M-12, J5 PJ301M-12, J6 PJ301M-12, Q3 2N3904, Q4 2N3904, SW1 SW_SPDT

Commit message: First print round
Changed lines of the file:
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@@
     (stroke (width 0) (type default))
   )
-  (wire (pts (xy 151.13 85.09) (xy 152.4 85.09))
+  (wire (pts (xy 151.13 80.01) (xy 152.4 80.01))
     (stroke (width 0) (type default))
   )
@@
     (stroke (width 0) (type default))
   )
-  (wire (pts (xy 151.13 85.09) (xy 151.13 86.36))
+  (wire (pts (xy 151.13 80.01) (xy 151.13 86.36))
     (stroke (width 0) (type default))
   )
@@
     (effects (font (size 1.27 1.27)) (justify left))
   )
-  (hierarchical_label "led 1 -" (shape input) (at 152.4 85.09 0) (fields_autoplaced)
+  (hierarchical_label "led 1 -" (shape input) (at 152.4 80.01 0) (fields_autoplaced)
     (effects (font (size 1.27 1.27)) (justify left))
   )
