File: circuit_panel.kicad_sch (KiCad schematic)
At the start: 47 parts, among them J1 Eurorack_Power_10pin_Unshroud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, Q1 2N3904, Q2 2N3904, Q5 2N3904, U1 TL074, U2 TL074

Commit message: First print round
Parts:
- added C4, C5: 1uF_0603_25V, Capacitor_THT:C_Disc_D3.8mm_W2.6mm_P2.50mm, symbol PCM_4ms_Capacitor:1uF_0603_25V
- added C6, C7: 10uf, Capacitor_THT:CP_Radial_D4.0mm_P2.00mm, symbol Device:C_Polarized
- C1: footprint Capacitor_THT:C_Axial_L3.8mm_D2.6mm_P7.50mm_Horizontal -> Capacitor_THT:C_Disc_D3.0mm_W1.6mm_P2.50mm
- C2: footprint Capacitor_THT:C_Disc_D3.8mm_W2.6mm_P2.50mm -> Capacitor_THT:C_Disc_D3.0mm_W1.6mm_P2.50mm
Connections:
- net +12V: now also C5.1, C7.1
- net -12V: now also C4.1, C6.2
- net GND: now also C4.2, C5.2, C6.1, C7.2
Changed lines of the file:
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@@
   (junction (at 109.22 82.55) (diameter 0) (color 0 0 0 0)
   )
+  (junction (at 35.56 50.8) (diameter 0) (color 0 0 0 0)
+  )
   (junction (at 22.86 66.04) (diameter 0) (color 0 0 0 0)
   )
@@
   (junction (at 92.71 57.15) (diameter 0) (color 0 0 0 0)
   )
+  (junction (at 35.56 82.55) (diameter 0) (color 0 0 0 0)
+  )
   (junction (at 204.47 74.93) (diameter 0) (color 0 0 0 0)
   )
@@
     (stroke (width 0) (type default))
   )
+  (wire (pts (xy 38.1 93.98) (xy 35.56 93.98))
+    (stroke (width 0) (type default))
+  )
   (wire (pts (xy 54.61 138.43) (xy 72.39 138.43))
     (stroke (width 0) (type default))
@@
     (stroke (width 0) (type default))
   )
+  (wire (pts (xy 35.56 93.98) (xy 35.56 82.55))
+    (stroke (width 0) (type default))
+  )
   (wire (pts (xy 251.46 82.55) (xy 251.46 86.36))
     (stroke (width 0) (type default))
@@
     (stroke (width 0) (type default))
   )
+  (wire (pts (xy 35.56 50.8) (xy 35.56 60.96))
+    (stroke (width 0) (type default))
+  )
   (wire (pts (xy 226.06 82.55) (xy 224.79 82.55))
     (stroke (width 0) (type default))
@@
     (stroke (width 0) (type default))
   )
+  (wire (pts (xy 35.56 82.55) (xy 36.83 82.55))
+    (stroke (width 0) (type default))
+  )
   (wire (pts (xy 168.91 46.99) (xy 168.91 58.42))
     (stroke (width 0) (type default))
@@
     (stroke (width 0) (type default))
   )
+  (wire (pts (xy 35.56 39.37) (xy 35.56 50.8))
+    (stroke (width 0) (type default))
+  )
   (wire (pts (xy 81.28 57.15) (xy 81.28 96.52))
     (stroke (width 0) (type default))
@@
     (stroke (width 0) (type default))
   )
+  (wire (pts (xy 43.18 50.8) (xy 46.99 50.8))
+    (stroke (width 0) (type default))
+  )
   (wire (pts (xy 92.71 57.15) (xy 97.79 57.15))
     (stroke (width 0) (type default))
@@
     (stroke (width 0) (type default))
   )
+  (wire (pts (xy 35.56 71.12) (xy 35.56 82.55))
+    (stroke (width 0) (type default))
+  )
   (wire (pts (xy 74.93 57.15) (xy 74.93 59.69))
     (stroke (width 0) (type default))
@@
     (stroke (width 0) (type default))
   )
+  (wire (pts (xy 35.56 39.37) (xy 36.83 39.37))
+    (stroke (width 0) (type default))
+  )
   (wire (pts (xy 172.72 121.92) (xy 179.07 121.92))
     (stroke (width 0) (type default))
@@
     (effects (font (size 1.27 1.27)) (justify left))
     (property "Intersheetrefs" "${INTERSHEET_REFS}" (at 50.8 102.3643 90)
+      (effects (font (size 1.27 1.27)) (justify left) hide)
+    )
+  )
+  (global_label "GND" (shape input) (at 44.45 82.55 0) (fields_autoplaced)
+    (effects (font (size 1.27 1.27)) (justify left))
+    (property "Intersheetrefs" "${INTERSHEET_REFS}" (at 51.3057 82.55 0)
       (effects (font (size 1.27 1.27)) (justify left) hide)
     )
@@
     )
   )
+  (global_label "GND" (shape input) (at 46.99 50.8 0) (fields_autoplaced)
+    (effects (font (size 1.27 1.27)) (justify left))
+    (property "Intersheetrefs" "${INTERSHEET_REFS}" (at 53.8457 50.8 0)
+      (effects (font (size 1.27 1.27)) (justify left) hide)
+    )
+  )
   (global_label "GND" (shape input) (at 172.72 69.85 270) (fields_autoplaced)
     (effects (font (size 1.27 1.27)) (justify right))
@@
     )
   )
+  (global_label "GND" (shape input) (at 43.18 93.98 0) (fields_autoplaced)
+    (effects (font (size 1.27 1.27)) (justify left))
+    (property "Intersheetrefs" "${INTERSHEET_REFS}" (at 50.0357 93.98 0)
+      (effects (font (size 1.27 1.27)) (justify left) hide)
+    )
+  )
   (global_label "GND" (shape input) (at 92.71 129.54 180) (fields_autoplaced)
     (effects (font (size 1.27 1.27)) (justify right))
@@
     )
   )
+  (global_label "GND" (shape input) (at 41.91 39.37 0) (fields_autoplaced)
+    (effects (font (size 1.27 1.27)) (justify left))
+    (property "Intersheetrefs" "${INTERSHEET_REFS}" (at 48.7657 39.37 0)
+      (effects (font (size 1.27 1.27)) (justify left) hide)
+    )
+  )
   (global_label "GND" (shape input) (at 111.76 80.01 0) (fields_autoplaced)
     (effects (font (size 1.27 1.27)) (justify left))
@@
         (path "/c67e14f9-c6f4-4089-b0b5-2e0894612a43/de5c4b79-7131-43bf-a16b-5b3b23a8530c"
           (reference "R20") (unit 1)
+        )
+      )
+    )
+  )
+  (symbol (lib_id "PCM_4ms_Capacitor:1uF_0603_25V") (at 39.37 39.37 90) (unit 1)
+    (in_bom yes) (on_board yes) (dnp no) (fields_autoplaced)
+    (property "Reference" "C5" (at 39.3763 33.02 90)
+      (effects (font (size 1.27 1.27)))
+    )
+    (property "Value" "1uF_0603_25V" (at 35.56 39.37 0)
+      (effects (font (size 1.27 1.27)) hide)
+    )
+    (property "Footprint" "Capacitor_THT:C_Disc_D3.8mm_W2.6mm_P2.50mm" (at 44.45 41.91 0)
+      (effects (font (size 1.27 1.27)) (justify left) hide)
+    )
+    (property "Datasheet" "" (at 39.37 39.37 0)
+      (effects (font (size 1.27 1.27)) hide)
+    )
+    (property "Specifications" "1uF, Min. 25V, 0603, Ceramic/MLCC" (at 47.244 41.91 0)
+      (effects (font (size 1.27 1.27)) (justify left) hide)
+    )
+    (property "Manufacturer" "Murata" (at 48.768 41.91 0)
+      (effects (font (size 1.27 1.27)) (justify left) hide)
+    )
+    (property "Part Number" "GRM188R61E105KA12D" (at 50.292 41.91 0)
+      (effects (font (size 1.27 1.27)) (justify left) hide)
+    )
+    (property "Display" "100nF/25V" (at 39.3763 35.56 90)
+      (effects (font (size 1.27 1.27)))
+    )
+    (property "JLCPCB ID" "C15849" (at 52.07 38.1 0)
+      (effects (font (size 1.27 1.27)) hide)
+    )
+    (pin "2")
+    (pin "1")
+    (instances
+      (project "ad-vca"
+        (path "/c67e14f9-c6f4-4089-b0b5-2e0894612a43/de5c4b79-7131-43bf-a16b-5b3b23a8530c"
+          (reference "C5") (unit 1)
         )
       )
@@
       (effects (font (size 1.27 1.27)) hide)
     )
-    (property "Footprint" "Capacitor_THT:C_Disc_D3.8mm_W2.6mm_P2.50mm" (at 170.18 72.39 0)
+    (property "Footprint" "Capacitor_THT:C_Disc_D3.0mm_W1.6mm_P2.50mm" (at 170.18 72.39 0)
       (effects (font (size 1.27 1.27)) (justify left) hide)
     )
@@
         (path "/c67e14f9-c6f4-4089-b0b5-2e0894612a43/de5c4b79-7131-43bf-a16b-5b3b23a8530c"
           (reference "R33") (unit 1)
+        )
+      )
+    )
+  )
+  (symbol (lib_id "Device:C_Polarized") (at 40.64 82.55 270) (unit 1)
+    (in_bom yes) (on_board yes) (dnp no) (fields_autoplaced)
+    (property "Reference" "C6" (at 41.529 74.93 90)
+      (effects (font (size 1.27 1.27)))
+    )
+    (property "Value" "10uf" (at 41.529 77.47 90)
+      (effects (font (size 1.27 1.27)))
+    )
+    (property "Footprint" "Capacitor_THT:CP_Radial_D4.0mm_P2.00mm" (at 36.83 83.5152 0)
+      (effects (font (size 1.27 1.27)) hide)
+    )
+    (property "Datasheet" "~" (at 40.64 82.55 0)
+      (effects (font (size 1.27 1.27)) hide)
+    )
+    (pin "2")
+    (pin "1")
+    (instances
+      (project "ad-vca"
+        (path "/c67e14f9-c6f4-4089-b0b5-2e0894612a43/de5c4b79-7131-43bf-a16b-5b3b23a8530c"
+          (reference "C6") (unit 1)
         )
       )
@@
     )
   )
+  (symbol (lib_id "PCM_4ms_Capacitor:1uF_0603_25V") (at 40.64 93.98 90) (unit 1)
+    (in_bom yes) (on_board yes) (dnp no) (fields_autoplaced)
+    (property "Reference" "C4" (at 40.6463 87.63 90)
+      (effects (font (size 1.27 1.27)))
+    )
+    (property "Value" "1uF_0603_25V" (at 36.83 93.98 0)
+      (effects (font (size 1.27 1.27)) hide)
+    )
+    (property "Footprint" "Capacitor_THT:C_Disc_D3.8mm_W2.6mm_P2.50mm" (at 45.72 96.52 0)
+      (effects (font (size 1.27 1.27)) (justify left) hide)
+    )
+    (property "Datasheet" "" (at 40.64 93.98 0)
+      (effects (font (size 1.27 1.27)) hide)
+    )
+    (property "Specifications" "1uF, Min. 25V, 0603, Ceramic/MLCC" (at 48.514 96.52 0)
+      (effects (font (size 1.27 1.27)) (justify left) hide)
+    )
+    (property "Manufacturer" "Murata" (at 50.038 96.52 0)
+      (effects (font (size 1.27 1.27)) (justify left) hide)
+    )
+    (property "Part Number" "GRM188R61E105KA12D" (at 51.562 96.52 0)
+      (effects (font (size 1.27 1.27)) (justify left) hide)
+    )
+    (property "Display" "100nf/25V" (at 40.6463 90.17 90)
+      (effects (font (size 1.27 1.27)))
+    )
+    (property "JLCPCB ID" "C15849" (at 53.34 92.71 0)
+      (effects (font (size 1.27 1.27)) hide)
+    )
+    (pin "2")
+    (pin "1")
+    (instances
+      (project "ad-vca"
+        (path "/c67e14f9-c6f4-4089-b0b5-2e0894612a43/de5c4b79-7131-43bf-a16b-5b3b23a8530c"
+          (reference "C4") (unit 1)
+        )
+      )
+    )
+  )
   (symbol (lib_id "Diode:1N4148") (at 101.6 57.15 0) (mirror y) (unit 1)
     (in_bom yes) (on_board yes) (dnp no)
@@
       (effects (font (size 1.27 1.27)) (justify left))
     )
-    (property "Value" "2N3904" (at 194.31 121.92 0)
+    (property "Value" "2N3904" (at 203.2 113.03 0)
       (effects (font (size 1.27 1.27)) (justify left))
     )
@@
       (effects (font (size 1.27 1.27)) hide)
     )
-    (property "Footprint" "Capacitor_THT:C_Axial_L3.8mm_D2.6mm_P7.50mm_Horizontal" (at 90.17 59.69 0)
+    (property "Footprint" "Capacitor_THT:C_Disc_D3.0mm_W1.6mm_P2.50mm" (at 90.17 59.69 0)
       (effects (font (size 1.27 1.27)) (justify left) hide)
     )
@@
         )
       )
+    )
+  )
+  (symbol (lib_id "Device:C_Polarized") (at 39.37 50.8 90) (unit 1)
+    (in_bom yes) (on_board yes) (dnp no) (fields_autoplaced)
+    (property "Reference" "C7" (at 38.481 43.18 90)
+      (effects (font (size 1.27 1.27)))
+    )
+    (property "Value" "10uf" (at 38.481 45.72 90)
+      (effects (font (size 1.27 1.27)))
+    )
+    (property "Footprint" "Capacitor_THT:CP_Radial_D4.0mm_P2.00mm" (at 43.18 49.8348 0)
+      (effects (font (size 1.27 1.27)) hide)
+    )
+    (property "Datasheet" "~" (at 39.37 50.8 0)
+      (effects (font (size 1.27 1.27)) hide)
+    )
+    (pin "2")
+    (pin "1")
+    (instances
+      (project "ad-vca"
+        (path "/c67e14f9-c6f4-4089-b0b5-2e0894612a43/de5c4b79-7131-43bf-a16b-5b3b23a8530c"
+          (reference "C7") (unit 1)
+        )
+      )

Commit message: Fixed bad tracing and reviewed circuit design
Parts:
- removed R20: 100k_0603, Resistor_THT:R_Axial_DIN0207_L6.3mm_D2.5mm_P7.62mm_Horizontal, symbol PCM_4ms_Resistor:100k_0603
- R23: Display 47k -> 4.7k
Connections:
- net lfo switch 1 is gone; now on net lfo led 1 -: R29.2
- net GND: no longer U1.12 (+)
- net adsr led 2 -: now also R3.1, R5.2, U1.6 (-), U1.7; no longer R15.1, R16.2, U2.14
- net lfo led 1 -: no longer R23.1, R24.1, R25.1
- net lfo pot 1: now also R23.1, R24.1, R25.1
- net at R6.2, R7.1, U1.9 (-): now also U1.13 (-)
- net at C1.1, R28.1, R29.1: now also U1.12 (+); no longer U1.13 (-)
- new net: R15.1, R16.2, U2.14
Other:
- moved on the sheet: R25
