File: control_panel.kicad_sch (KiCad schematic)
At the start: 17 parts, among them J3 PJ301M-12, J4 PJ301M-12, J5 PJ301M-12, J6 PJ301M-12, Q3 2N3904, Q4 2N3904, SW1 SW_SPDT

Commit message: Fixed bad tracing and reviewed circuit design
Connections:
- net Audio In: now also J3.3; no longer J3.1
- net Audio Out: now also J4.3; no longer J4.1
- net Cv out: now also J5.3; no longer J5.1
- net GND: now also J3.1, J4.1, J5.1, J6.1; no longer J3.3, J4.3, J5.3, J6.3
- net Gate In: now also J6.3; no longer J6.1
- net led 1 +: now also D6.2 (A); no longer R26.1
- net led 1 -: now also R30.1; no longer D7.1 (K)
- net led 2 +: now also D7.2 (A); no longer R30.1
- net led 2 -: now also R26.1; no longer D6.1 (K)
- net at Q4.3 (C): now also D6.1 (K); no longer D6.2 (A)
- net at Q3.3 (C): now also D7.1 (K); no longer D7.2 (A)
Other:
- moved on the sheet: D6, D7, R26
